Commit message: WSL sim support, CCW spiral toolpath, Nav2 tuning for coverage mowing
Major changes:
- Rewrote strip_generator.py: headland pattern → CCW inward spiral
  (mower discharges right, spiral keeps clippings inward)
- Waypoint spacing reduced 5m→1.5m for smooth controller tracking
- mission_node.py: added transit path generation, TF readiness checks,
  radio evacuation support, /fromLL coordinate conversion
- Gazebo world: exact polygon boundary from RTK survey via /fromLL
  (4 edge lines + 4 red corner cubes replace approximate rectangle)
- Aligned Gazebo spherical_coordinates origin with navsat datum
  (50.63447, -105.03184) to eliminate coordinate system mismatch
- sim.launch.py: park position spawn, odom kickstart, IMU relay,
  magnetic declination override for sim
- Nav2 RPP tuning: curvature-based slowing, collision detection off,
  500m pose search for 5000m spiral path, generous progress checker
- Added scripts/sim_imu_relay.py to bridge Gazebo IMU → localization
- Added utils/wsl-setup.sh and Makefile targets for WSL workflow
  (rsync, colcon build, sim launch — alternative to Docker)

Known issues (documented in sim-tuning.md):
- Controller aborts at tight spiral corners (~0.76m radius)
- Consistent ~5m westward path tracking offset under investigation
- Gazebo NavSat publishes zero covariance (may affect EKF fusion)

Co-Authored-By: Claude Opus 4.6 <noreply@anthropic.com>

File: description/imu.xacro (robot description, xacro)
@@ -1,4 +1,5 @@
 <?xml version="1.0"?>
 <robot xmlns:xacro="http://www.ros.org/wiki/xacro" name="imu">
+    <!-- IMU TF frame — needed by robot_localization -->
     <joint name="imu_joint" type="fixed">
         <parent link="base_link"/>
@@ -7,15 +8,23 @@
     </joint>
     <link name="imu">
+        <visual>
+            <geometry>
+                <box size="0.02 0.02 0.005"/>
+            </geometry>
+            <material name="imu_grey">
+                <color rgba="0.4 0.4 0.4 1"/>
+            </material>
+        </visual>
     </link>
-    <gazebo reference="imu">
-        <sensor name="imu" type="imu">
+    <!-- Sensor attached to base_link so it survives URDF→SDF fixed-joint merging.
+         The imu link above still provides the TF frame for robot_localization. -->
+    <gazebo reference="base_link">
+        <sensor name="imu_sensor" type="imu">
             <gz_frame_id>imu</gz_frame_id>
-            <!-- not possible to disable orientation via SDF, we will skip it during fusion-->
             <always_on>1</always_on>
             <update_rate>50</update_rate>
-            <visualize>true</visualize>
             <topic>imu/data_raw</topic>
+            <pose>${robot['imu']['chip']['offset'][0]} ${robot['imu']['chip']['offset'][1]} ${robot['imu']['chip']['offset'][2]} 0 0 0</pose>
         </sensor>
-        <material>Gazebo/Red</material>
     </gazebo>
 </robot>

File: description/robot.urdf.xacro (robot description, xacro)
@@ -7,4 +7,5 @@
     <xacro:include filename="robot_core.xacro" />
     <xacro:include filename="gps.xacro" />
+    <xacro:include filename="imu.xacro" />
     <xacro:if value="$(arg use_ros2_control)">
         <xacro:include filename="ros2_control.xacro" />
