File: hardware/moxl-hat/moxl-hat.kicad_pcb (KiCad board)
At the start: 6 copper layers, 65 x 56 mm, 86 parts, among them J1 12V, J10 GPIO, J11 RS232, J2 CAN, J3 Left Motor, J4 Right Motor, J5 Relay Drivers, J6 Conn_01x08_Pin, J7 Analog Sense, J8 Conn_01x03_Pin, J9 Thermo, U1 MAX31855KASA, U10 74HC14D,653, U12 TPS7A7001DDA, U15 XL4015, U2 TLP293-4, U3 ADS1115IDGS, U4 TLP293-4, U5 MCP251863T-E/SSVAO, U6 PCA9685PW, U7 ULN2003A, U8 CAT24C256, U9 MAX3221EIPWR, Y1 20Mhz

Commit message: Mo-XL Hat v1.0: clean DRC schematic/PCB, spec sheet, JLCPCB production files
- Schematic and PCB pass DRC clean, 6-layer ENIG stackup
- J3/J4 changed from JST-XH to 2x4 IDC headers (ribbon cable to BTS7960)
- CAT24C256 EEPROM populated (not DNP)
- Added pinout-table.dxf for bottom silk layer (GPIO map + connector pinouts)
- Added gen_pinout_dxf.py and gen_spec_pdf.py generators
- Spec sheet PDF: features, BOM, GPIO map, connectors, trace widths,
  power architecture, engine control, schematic appendix
- JLCPCB production files: BOM, positions, netlist, Gerber zip
- Updated HARDWARE_TODO and hat spec for IDC connectors, encoder inputs

Co-Authored-By: Claude Opus 4.6 <noreply@anthropic.com>
Parts:
- removed C24: 220uF/50V, Capacitor_SMD:CP_Elec_10x10.5
- removed C28: 330uF/25V, Capacitor_SMD:CP_Elec_10x10.5
- removed D2: TPSMB18A, Diode_SMD:D_SMB
- removed R21: 0, Resistor_SMD:R_0402_1005Metric
- removed R33: 10k, Resistor_SMD:R_0603_1608Metric
- added C18: 47uF/25V, Capacitor_SMD:C_1210_3225Metric, F.Cu at (117.5, 86.0)
- added C20: 47uF/25V, Capacitor_SMD:C_1210_3225Metric, F.Cu at (125.0, 67.7)
- added C21: 47uF/25V, Capacitor_SMD:C_1210_3225Metric, F.Cu at (124.9, 71.0)
- added C9: 47uF/25V, Capacitor_SMD:C_1210_3225Metric, F.Cu at (117.5, 89.4)
- added F1: 3A, Fuse:Fuse_1812_4532Metric, F.Cu at (124.6, 98.0)
- added F2: 200mA, Fuse:Fuse_0805_2012Metric, F.Cu at (111.8, 92.5)
- added J12: Conn_01x03_Pin, Connector_JST:JST_PH_B3B-PH-K_1x03_P2.00mm_Vertical, F.Cu at (132.6, 52.6)
- added R26: 30.1K, PCM_JLCPCB:R_0603, F.Cu at (122.4, 57.3)
- added R27: 274K, PCM_JLCPCB:R_0603, F.Cu at (125.1, 57.3)
- added R28: 10kΩ, PCM_JLCPCB:R_0603, F.Cu at (123.0, 73.5)
- added TP3: 3V3, TestPoint:TestPoint_THTPad_D1.5mm_Drill0.7mm, F.Cu at (161.4, 91.5)
- C19: footprint Capacitor_SMD:C_0603_1608Metric -> PCM_JLCPCB:C_0603
- C3, JP1, U8: moved to F.Cu
- C6: value 100n -> .1uF; moved to F.Cu
- J3, J4: footprint Connector_JST:JST_XH_B6B-XH-A_1x06_P2.50mm_Vertical -> Connector_PinHeader_2.54mm:PinHeader_2x04_P2.54mm_Vertical
- J8: value Conn_01x03_Pin -> Pulse_Inputs; footprint Connector_JST:JST_XH_B3B-XH-A_1x03_P2.50mm_Vertical -> Connector_JST:JST_PH_B5B-PH-K_1x05_P2.00mm_Vertical
- J9: value Thermo -> CHT_Type_K
- L4: value 47uH/5A -> 33uH/4A; footprint Inductor_SMD:L_Sunlord_MWSA1206S-470 -> Inductor_SMD:L_Changjiang_FXL1040
- R19, R20: value 0 -> 0Ω; footprint Resistor_SMD:R_0402_1005Metric -> PCM_JLCPCB:R_0603
- R2, R3: value 3.9k -> 3.9kΩ; footprint Resistor_SMD:R_0402_1005Metric -> PCM_JLCPCB:R_0402; moved to F.Cu
- moved TP2 91.9 mm to (161.4, 85.9)
- moved C11 83.4 mm to (157.5, 89.9), turned to 90 degrees
- moved R25 74.8 mm to (141.0, 78.0), turned to 90 degrees
- moved J11 73.2 mm to (141.6, 52.6)
- moved C7 68.6 mm to (119.0, 93.3)
- moved C8 67.8 mm to (121.7, 86.8)
- moved C27 65.2 mm to (119.5, 62.6)
- moved TP1 63.0 mm to (133.5, 72.8)
- moved C26 62.5 mm to (118.8, 82.6), turned to -90 degrees
- moved C25 60.8 mm to (116.7, 82.6), turned to -90 degrees
- moved TP7 58.8 mm to (129.2, 72.5)
- moved R20 58.3 mm to (118.8, 57.9)
- moved TP6 56.7 mm to (126.0, 87.3)
- moved C10 56.6 mm to (136.2, 71.2), turned to -90 degrees
- moved U10 54.8 mm to (134.5, 61.3)
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Connections:
- net 12-28V renamed Net-(C7-Pad2)
- C25 pad 2: Net-(U15-VIN) -> +12V
- C26 pad 2: Net-(U15-VIN) -> +12V
- C8 pad 1: /12V -> +12V
- D1 pad 1: /12V -> +12V
- D1 pad 2: Net-(D1-A2) -> GND
- J1 pad 1: Net-(J1-Pin_1) -> GND
- J1 pad 2: GND -> /12V_Raw
- J10 pad 29: /GPIO5 -> /GPIO5_Relay_Aux
- J3 pad 5: +5V -> unconnected-(J3-Pin_5-Pad5)
- J3 pad 6: GND -> unconnected-(J3-Pin_6-Pad6)
- J4 pad 5: +5V -> unconnected-(J4-Pin_5-Pad5)
- J4 pad 6: GND -> unconnected-(J4-Pin_6-Pad6)
- J7 pad 3: /FUEL -> /FUEL_LEVEL
- J8 pad 2: +5V -> /ENC_L
- J8 pad 3: GND -> /ENC_R
- L1 pad 2: /12V -> +12V
- R19 pad 1: /GPIO14/TXD0 -> /GPIO15/RXD0
- R19 pad 2: /Uart_Din -> /Uart_Dout
- R20 pad 2: /Uart_Dout -> /SBUS
- TP6 pad 1: Net-(U15-VIN) -> +12V
- U10 pad 5: GND -> /ENC_L
- U10 pad 6: unconnected-(U10-3Y-Pad6) -> /GPIO6
- U10 pad 8: unconnected-(U10-4Y-Pad8) -> /GPIO19/PCM.FS
- U10 pad 9: GND -> /ENC_R
- U15 pad 5: Net-(U15-VIN) -> +12V
- U3 pad 1: unconnected-(U3-ADDR-Pad1) -> GND
- U7 pad 4: unconnected-(U7-I4-Pad4) -> /GPIO5_Relay_Aux
- U7 pad 5: unconnected-(U7-I5-Pad5) -> GND
- U7 pad 6: unconnected-(U7-I6-Pad6) -> GND
- U7 pad 7: unconnected-(U7-I7-Pad7) -> GND
- U7 pad 8: unconnected-(U7-GND-Pad8) -> GND
- U7 pad 9: unconnected-(U7-COM-Pad9) -> +12V
- U9 pad 11: /Uart_Din -> /GPIO14/TXD0
Routing:
- net GND: track 0.00 -> 72.9 mm, vias 0 -> 40
- net /I2C_SDA: track 0.00 -> 69.3 mm, vias 0 -> 3
- net /I2C_SCL: track 0.00 -> 68.9 mm, vias 0 -> 3
- net /SPI_SCK: track 0.00 -> 66.4 mm, vias 0 -> 3
- net /SPI_MISO: track 0.00 -> 64.6 mm, vias 0 -> 3
- net /SPI_CS1_TC: track 0.00 -> 60.1 mm, vias 0 -> 3
- net /CAN_INT: track 0.00 -> 55.8 mm, vias 0 -> 5
- net +12V: track 0.00 -> 55.5 mm, vias 0 -> 2
- net +6V: track 0.00 -> 54.8 mm
- net /SPI_MOSI: track 0.00 -> 54.6 mm, vias 0 -> 3
- net /SPI_CS0_CAN: track 0.00 -> 51.8 mm, vias 0 -> 3
- net /SERVO_CHKTHRTL: track 0.00 -> 50.6 mm, vias 0 -> 2
- net /SERVO1: track 0.00 -> 48.8 mm, vias 0 -> 2
- net +3V3: track 0.00 -> 48.0 mm, vias 0 -> 12
- net /SERVO2: track 0.00 -> 46.6 mm, vias 0 -> 2
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- added copper zone on F.Cu, net +12V
- added copper zone on In2.Cu, net +3V3
- added copper zone on F.Cu, net +5V
- added copper zone on In2.Cu, net +5V
- added copper zone on F.Cu, net +6V
- added copper zone on F.Cu, net /12V_Raw
- added copper zone on B.Cu, net GND
- added copper zone on F.Cu, net GND
- added copper zone on In1.Cu, net GND
- added copper zone on In3.Cu, net GND
- added copper zone on In4.Cu, net GND
- added copper zone on F.Cu, net Net-(C7-Pad2)
- added copper zone on F.Cu, net Net-(D13-K)
Other:
- outline, holes or cut-outs redrawn
- board text added: "Mo-XL v1.0"
- board text added: "Rx232"
- board text added: "SBUS"
- board text removed: "Extend PCB edge 0.5mm if using SMT header"
