File: hardware/moxl-hat/moxl-hat.kicad_sch (KiCad schematic)
At the start: 86 parts, among them J1 12V, J10 GPIO, J11 RS232, J2 CAN, J3 Left Motor, J4 Right Motor, J5 Relay Drivers, J6 Conn_01x08_Pin, J7 Analog Sense, J8 Conn_01x03_Pin, J9 Thermo, U1 MAX31855KASA, U10 74HC14D,653, U12 TPS7A7001DDA, U15 XL4015, U2 TLP293-4, U3 ADS1115IDGS, U4 TLP293-4, U5 MCP251863T-E/SSVAO, U6 PCA9685PW, U7 ULN2003A, U8 CAT24C256, U9 MAX3221EIPWR, Y1 20Mhz

Commit message: Mo-XL Hat v1.0: clean DRC schematic/PCB, spec sheet, JLCPCB production files
- Schematic and PCB pass DRC clean, 6-layer ENIG stackup
- J3/J4 changed from JST-XH to 2x4 IDC headers (ribbon cable to BTS7960)
- CAT24C256 EEPROM populated (not DNP)
- Added pinout-table.dxf for bottom silk layer (GPIO map + connector pinouts)
- Added gen_pinout_dxf.py and gen_spec_pdf.py generators
- Spec sheet PDF: features, BOM, GPIO map, connectors, trace widths,
  power architecture, engine control, schematic appendix
- JLCPCB production files: BOM, positions, netlist, Gerber zip
- Updated HARDWARE_TODO and hat spec for IDC connectors, encoder inputs

Co-Authored-By: Claude Opus 4.6 <noreply@anthropic.com>
Parts:
- removed C19: 10uF, Capacitor_SMD:C_0603_1608Metric, symbol ESP32-S3 TFT Touch v1.1(3.5'' ili9488)-eagle-import:C-0603
- removed C24: 220uF/50V, Capacitor_SMD:CP_Elec_10x10.5, symbol Device:C_Polarized_Small_US
- removed C28: 330uF/25V, Capacitor_SMD:CP_Elec_10x10.5, symbol Device:C_Polarized_Small_US
- removed D2: TPSMB18A, Diode_SMD:D_SMB, symbol troo:D_TVS_Single
- removed J3: Left Motor, Connector_JST:JST_XH_B6B-XH-A_1x06_P2.50mm_Vertical, symbol Connector:Conn_01x06_Pin
- removed J4: Right Motor, Connector_JST:JST_XH_B6B-XH-A_1x06_P2.50mm_Vertical, symbol Connector:Conn_01x06_Pin
- removed J8: Conn_01x03_Pin, Connector_JST:JST_XH_B3B-XH-A_1x03_P2.50mm_Vertical, symbol Connector:Conn_01x03_Pin
- removed R19, R20, R21: 0, Resistor_SMD:R_0402_1005Metric, symbol Device:R_Small
- removed R2, R3: 3.9k, Resistor_SMD:R_0402_1005Metric, symbol Device:R_Small
- removed R33: 10k, Resistor_SMD:R_0603_1608Metric, symbol jlcpcb-basic-resistor:0603,10k
- added C18, C20, C21, C9: 47uF/25V, Capacitor_SMD:C_1210_3225Metric, symbol Device:C_Small
- added C19: 10uF, PCM_JLCPCB:C_0603, symbol PCM_JLCPCB-Capacitors:0603,10uF
- added J12: Conn_01x03_Pin, Connector_JST:JST_PH_B3B-PH-K_1x03_P2.00mm_Vertical, symbol Connector:Conn_01x03_Pin
- added J3: Left Motor, Connector_PinHeader_2.54mm:PinHeader_2x04_P2.54mm_Vertical, symbol Connector_Generic:Conn_02x04_Odd_Even
- added J4: Right Motor, Connector_PinHeader_2.54mm:PinHeader_2x04_P2.54mm_Vertical, symbol Connector_Generic:Conn_02x04_Odd_Even
- added J8: Pulse_Inputs, Connector_JST:JST_PH_B5B-PH-K_1x05_P2.00mm_Vertical, symbol Connector:Conn_01x05_Pin
- added R19, R20: 0Ω, PCM_JLCPCB:R_0603, symbol PCM_JLCPCB-Resistors:0603,0Ω
- added R2, R3: 3.9kΩ, PCM_JLCPCB:R_0402, symbol PCM_JLCPCB-Resistors:0402,3.9kΩ
- added R28: 10kΩ, PCM_JLCPCB:R_0603, symbol PCM_JLCPCB-Resistors:0603,10kΩ
- added TP3: 3V3, TestPoint:TestPoint_THTPad_D1.5mm_Drill0.7mm, symbol Connector:TestPoint
- C6: value 100n -> .1uF; LCSC (none) -> C14663; now fitted
- F1: value 2A -> 3A; footprint (none) -> Fuse:Fuse_1812_4532Metric; LCSC (none) -> C20627123
- F2: footprint (none) -> Fuse:Fuse_0805_2012Metric; LCSC (none) -> C20976
- J1: LCSC (none) -> C495202
- J11: LCSC (none) -> C131339
- J2: LCSC (none) -> C594232
- J5: LCSC (none) -> C157991
- J6: LCSC (none) -> C157972
- J7: LCSC (none) -> C157993
- J9: value Thermo -> CHT_Type_K; LCSC (none) -> C158012
- JP1: now fitted
- L4: value 47uH/5A -> 33uH/4A; footprint Inductor_SMD:L_Sunlord_MWSA1206S-470 -> Inductor_SMD:L_Changjiang_FXL1040; LCSC C408531 -> C436575
- R26: footprint (none) -> PCM_JLCPCB:R_0603; LCSC (none) -> C23000
- R27: footprint (none) -> PCM_JLCPCB:R_0603; LCSC (none) -> C22968
- U1: LCSC (none) -> C52028
- U12: LCSC (none) -> C60719
- U2, U4: LCSC (none) -> C112623
- U3: LCSC C37593 -> C2868291
- U6: LCSC (none) -> C2678753
- U7: LCSC (none) -> C482013
- U8: LCSC (none) -> C79987; now fitted
Connections:
- net 12V is gone; now on net +12V: C8.1, D1.1 (A1), L1.2
- net FUEL is gone; now on net FUEL_LEVEL: J7.3 (Pin_3)
- net GPIO5 is gone; now on net GPIO5_Relay_Aux: J10.29 (Pin_29)
- net Uart_Din is gone; now on net GPIO14/TXD0: U9.11 (DIN)
- net +12V: now also C25.2, C26.2, TP6.1, U15.5 (VIN), U7.9 (COM), C18.1, C9.1; no longer F1.1
- net +3V3: now also R2.1, R3.1, TP3.1
- net +5V: now also C19.1, J12.2 (Pin_2), J3.7 (Pin_7), J4.7 (Pin_7), J8.4 (Pin_4)
- net +6V: now also C20.1, C21.1, R28.1
- net BTS_L_LEN: now also J3.4 (Pin_4)
- net BTS_L_LPWM: now also J3.2 (Pin_2)
- net BTS_L_REN: now also J3.3 (Pin_3)
- net BTS_L_RPWM: now also J3.1 (Pin_1)
- net BTS_R_LEN: now also J4.4 (Pin_4)
- net BTS_R_LPWM: now also J4.2 (Pin_2)
- net BTS_R_REN: now also J4.3 (Pin_3)
- net BTS_R_RPWM: now also J4.1 (Pin_1)
- net GND: now also D1.2 (A2), J1.1 (Pin_1), U3.1 (ADDR), U7.5 (I5), U7.6 (I6), U7.7 (I7), U7.8 (GND), C18.2, C19.2, C20.2, C21.2, C9.2, J12.3 (Pin_3), J3.8 (Pin_8), J4.8 (Pin_8), J8.5 (Pin_5); no longer J1.2 (Pin_2), U10.5 (3A), U10.9 (4A)
- net GPIO15/RXD0: now also R19.1, R20.1
- net GPIO19/PCM.FS: now also U10.8 (4Y)
- net GPIO6: now also U10.6 (3Y)
- net ID_SCL: now also R3.2
- net ID_SDA: now also R2.2
- net SBUS: now also R20.2
- net SBUS_FRSKY: now also J12.1 (Pin_1)
- net TACH: now also J8.1 (Pin_1)
- net Uart_Dout: now also R19.2
- net GPIO5_Relay_Aux: now reaches U7.4 (I4)
- net at R24.1, U15.2 (FB): now also R28.2
- net 12V_Raw: now reaches F1.2
- net 12V_Raw: now also J1.2 (Pin_2); no longer J1.1 (Pin_1)
- net 12-28V: no longer names the net of C7.2, L1.1
- net 12-28V: now also F1.1
- new net ENC_L: J8.2 (Pin_2), U10.5 (3A)
- new net ENC_R: J8.3 (Pin_3), U10.9 (4A)
- no-connect marks 23 -> 30
Other:
- note added: "EMI/TVS"
- note added: "SECTION: ANALOG SENSING ADS1115: I2C 16-bit ADC @ addr 0x48 AIN0: Battery 12V (Bottom 12V Bat) AIN1: Alternator current (ACS712 or shunt) AIN2: Fuel level (resistive float sender) AIN3: Battery Pack 24V (12V+12V)"
- note removed: "BATT_V, ALT_I, FUEL, SPARE_A"
- note removed: "SECTION: ANALOG SENSING ADS1115: I2C 16-bit ADC @ addr 0x48 AIN0: Battery 12V (Bottom 12V Bat) AIN1: Alternator current (ACS712 or shunt) AIN2: Fuel level (resistive float sender) AIN3: Battery Pack 24V (12V+12V) ADDR pin to GND for addr 0x48"
- note removed: "SECTION: POWER NOT SHOWN — add separately: 24V input → LMR36520 buck → 5V/2A (Pi power) 24V input → isolated DC-DC → 3.3V (opto field side) 6V regulator for servo power rail Input protection: TVS + reverse polarity MOSFET Resettable fuse on 24V input"
- note removed: "SECTION: RPM TACH INPUT NOT SHOWN — add separately: GPIO4 ← Schmitt trigger (74HC14) ← opto-isolator ← tach sensor Pullup on sensor side, series resistor for LED drive"
- note removed: "TODO: Replace all symbols with JLCPCB library equivalents TODO: Add Pi 40-pin GPIO header connector TODO: Add all external connectors (CAN, motors, servos, analog, TC, power) TODO: Add decoupling capacitors (100nF on every IC VCC) TODO: Add 40MHz crystal for MCP251863T TODO: Add LED current limiting resistors (330R) for opto-isolators TODO: Add voltage divider for battery sense (100K/33K) TODO: A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"
- title: (none) -> Mo-XL Pi Hat
- moved on the sheet: C7, C8, D1, F1, J1, J2, L1, R24
